Commit message: update kinova control

File: Robots/hand/robots/robotiq_arg85_description.urdf (robot description, URDF)
Before this commit: robot robotiq_arg85_description, 9 links, 8 joints
Joints:
- removed joint finger_joint
- added joint left_outer_knuckle_joint: type revolute, parent robotiq_85_base_link, child left_outer_knuckle, origin xyz=0.0306011444260539 0 0.0627920162695395 rpy=0 0 0, axis 0 -1 0, limit lower=0 upper=0.725 effort=1000 velocity=2.0
