Commit message: linked hand

File: Robots/gen3/6dof/urdf/GEN3_Hand.urdf (robot description, URDF)
Before this commit: robot GEN3-6DOF_VISION_URDF_ARM_V01, 8 links, 7 joints
Links:
- removed link EndEffector_Link
- added link left_inner_finger, mass 0.00724255346165745; collision mesh filename=package://gen3/6dof/meshes/inner_finger_coarse.STL; visual mesh filename=package://gen3/6dof/meshes/inner_finger_fine.STL
- added link left_inner_knuckle, mass 0.0110930853895903; collision mesh filename=package://gen3/6dof/meshes/inner_knuckle_coarse.STL; visual mesh filename=package://gen3/6dof/meshes/inner_knuckle_fine.STL
- added link left_outer_finger, mass 0.0273093985570947; collision mesh filename=package://gen3/6dof/meshes/outer_finger_coarse.STL; visual mesh filename=package://gen3/6dof/meshes/outer_finger_fine.STL
- added link left_outer_knuckle, mass 0.00684838849434396; collision mesh filename=package://gen3/6dof/meshes/outer_knuckle_coarse.STL; visual mesh filename=package://gen3/6dof/meshes/outer_knuckle_fine.STL
- added link right_inner_finger, mass 0.00724255346165744; collision mesh filename=package://gen3/6dof/meshes/inner_finger_coarse.STL; visual mesh filename=package://gen3/6dof/meshes/inner_finger_fine.STL
- added link right_inner_knuckle, mass 0.0110930853895903; collision mesh filename=package://gen3/6dof/meshes/inner_knuckle_coarse.STL; visual mesh filename=package://gen3/6dof/meshes/inner_knuckle_fine.STL
- added link right_outer_finger, mass 0.0273093985570947; collision mesh filename=package://gen3/6dof/meshes/outer_finger_coarse.STL; visual mesh filename=package://gen3/6dof/meshes/outer_finger_fine.STL
- added link right_outer_knuckle, mass 0.00684838849401352; collision mesh filename=package://gen3/6dof/meshes/outer_knuckle_coarse.STL; visual mesh filename=package://gen3/6dof/meshes/outer_knuckle_fine.STL
- added link robotiq_85_base_link, mass 0.30915; collision mesh filename=package://gen3/6dof/meshes/robotiq_85_base_link_coarse.STL; visual mesh filename=package://gen3/6dof/meshes/robotiq_85_base_link_fine.STL
Joints:
- added joint finger_joint: type revolute, parent robotiq_85_base_link, child left_outer_knuckle, origin xyz=0.0306011444260539 0 0.0627920162695395 rpy=0 0 0, axis 0 -1 0, limit lower=0 upper=0.725 effort=1000 velocity=2.0
- added joint left_inner_finger_joint: type revolute, parent left_inner_knuckle, child left_inner_finger, origin xyz=0.034585310861294 0 0.0454970193817975 rpy=0 0 0, axis 0 -1 0, limit lower=0 upper=0.8757 effort=1000 velocity=2.0, mimic joint=finger_joint multiplier=-1 offset=0
- added joint left_inner_knuckle_joint: type revolute, parent robotiq_85_base_link, child left_inner_knuckle, origin xyz=0.0127000000001501 0 0.0693074999999639 rpy=0 0 0, axis 0 -1 0, limit lower=0 upper=0.8757 effort=1000 velocity=2.0, mimic joint=finger_joint multiplier=1 offset=0
- added joint left_outer_finger_joint: type fixed, parent left_outer_knuckle, child left_outer_finger, origin xyz=0.0316910442266543 0 -0.00193396375724605 rpy=0 0 0, axis 0 -1 0
- added joint right_inner_finger_joint: type revolute, parent right_inner_knuckle, child right_inner_finger, origin xyz=0.0341060475457406 0 0.0458573878541688 rpy=0 0 0, axis 0 1 0, limit lower=0 upper=0.8757 effort=1000 velocity=2.0, mimic joint=finger_joint multiplier=1 offset=0
- added joint right_inner_knuckle_joint: type revolute, parent robotiq_85_base_link, child right_inner_knuckle, origin xyz=-0.0126999999998499 0 0.0693075000000361 rpy=0 0 3.14159265358979, axis 0 1 0, limit lower=0 upper=0.8757 effort=1000 velocity=2.0, mimic joint=finger_joint multiplier=-1 offset=0
- added joint right_outer_finger_joint: type fixed, parent right_outer_knuckle, child right_outer_finger, origin xyz=0.0317095909367246 0 -0.0016013564954687 rpy=0 0 0, axis 0 1 0
- added joint right_outer_knuckle_joint: type revolute, parent robotiq_85_base_link, child right_outer_knuckle, origin xyz=-0.0306011444258893 0 0.0627920162695395 rpy=0 0 3.14159265358979, axis 0 1 0, limit lower=0 upper=0.8757 effort=1000 velocity=2.0, mimic joint=finger_joint multiplier=-1 offset=0
- joint EndEffector: child EndEffector_Link -> robotiq_85_base_link

Commit message: update fingers

File: Robots/gen3/6dof/urdf/GEN3_Hand.urdf (robot description, URDF)
Before this commit: robot GEN3-6DOF_VISION_URDF_ARM_V01, 16 links, 15 joints
Joints:
- joint left_inner_finger_joint: limit lower=0 upper=0.8757 effort=1000 velocity=2.0 -> lower=-0.8757 upper=0 effort=1000 velocity=2.0
- joint right_inner_knuckle_joint: limit lower=0 upper=0.8757 effort=1000 velocity=2.0 -> lower=-0.8757 upper=0 effort=1000 velocity=2.0
- joint right_outer_knuckle_joint: limit lower=0 upper=0.8757 effort=1000 velocity=2.0 -> lower=-0.8757 upper=0 effort=1000 velocity=2.0
